File: diseños-3d/stick-pcb/stick-pcb.kicad_sch (KiCad schematic)
At the start: 32 parts, among them J1 Conn_01x05, J10 Conn_01x02, J11 Conn_01x02, J12 Conn_01x02, J13 Conn_01x02, J14 Conn_01x02, J15 Conn_01x02, J16 Conn_01x02, J17 Conn_01x02, J18 Conn_01x02, J19 Conn_01x02, J2 Conn_01x02, J20 Conn_01x02, J21 Conn_01x02, J22 Conn_01x02, J23 Conn_01x02, J3 Conn_01x02, J4 Conn_01x02, J5 Conn_01x02, J6 Conn_01x02, J7 Conn_01x02, J8 Conn_01x02, J9 Conn_01x02, U1 4021, U2 4021, U3 4021

Commit message: añadidas imágenes a la guía de GitHub
Parts:
- added J24, J25: Conn_01x02, Connector_PinHeader_2.54mm:PinHeader_1x02_P2.54mm_Vertical, symbol Connector_Generic:Conn_01x02
Connections:
- net GND: now also J24.1 (Pin_1), J25.2 (Pin_2)
- net Bit7: now reaches J15.2 (Pin_2)
- net Bit7: now also RN1.2 (R1), U1.1 (D7)
- net Bit10: now reaches J22.2 (Pin_2)
- net Bit10: now also RN2.7 (R6), U2.5 (D2)
- net Bit15: now reaches J12.1 (Pin_1)
- net Bit15: now also RN2.2 (R1), U2.1 (D7)
- net Bit18: now reaches J17.1 (Pin_1)
- net Bit18: now also RN3.7 (R6), U3.5 (D2)
- net Bit0: now reaches J2.2 (Pin_2)
- net Bit0: now also RN1.9 (R8), U1.7 (D0)
- net Bit21: now reaches J23.1 (Pin_1)
- net Bit21: now also RN3.4 (R3), U3.14 (D5)
- net Bit12: now reaches J5.1 (Pin_1)
- net Bit12: now also RN2.5 (R4), U2.13 (D4)
- net Bit4: now reaches J10.2 (Pin_2)
- net Bit4: now also RN1.5 (R4), U1.13 (D4)
- net Bit2: now reaches J6.2 (Pin_2)
- net Bit2: now also RN1.7 (R6), U1.5 (D2)
- net Bit16: now reaches J13.1 (Pin_1)
- net Bit16: now also RN3.9 (R8), U3.7 (D0)
- net Bit5: now reaches J11.2 (Pin_2)
- net Bit5: now also RN1.4 (R3), U1.14 (D5)
- net Bit13: now reaches U2.14 (D5)
- net Bit13: now also J8.1 (Pin_1), RN2.4 (R3)
- net Bit14: now reaches U2.15 (D6)
- net Bit14: now also J9.1 (Pin_1), RN2.3 (R2)
- net Bit11: now reaches U2.4 (D3)
- net Bit11: now also J3.1 (Pin_1), RN2.6 (R5)
- net Bit9: now reaches U2.6 (D1)
- net Bit9: now also J19.2 (Pin_2), RN2.8 (R7)
- net Bit8: now reaches U2.7 (D0)
- net Bit8: now also J18.2 (Pin_2), RN2.9 (R8)
- net Bit17: now reaches J16.1 (Pin_1)
- net Bit17: now also RN3.8 (R7), U3.6 (D1)
- net Bit20: now reaches J21.1 (Pin_1)
- net Bit20: now also RN3.5 (R4), U3.13 (D4)
- net Bit23: now reaches U3.1 (D7)
- net Bit23: now also RN3.2 (R1), J25.1 (Pin_1)
- net Bit22: now reaches U3.15 (D6)
- net Bit22: now also RN3.3 (R2), J24.2 (Pin_2)
- net Bit19: now reaches U3.4 (D3)
- net Bit19: now also J20.1 (Pin_1), RN3.6 (R5)
- net Bit6: now reaches RN1.3 (R2)
- net Bit6: now also J14.2 (Pin_2), U1.15 (D6)
- net Bit3: now reaches RN1.6 (R5)
- net Bit3: now also J7.2 (Pin_2), U1.4 (D3)
- net Bit1: now reaches RN1.8 (R7)
- net Bit1: now also J4.2 (Pin_2), U1.6 (D1)
Other:
- moved on the sheet: J11, J13, J14, J15, J16, J17, J18, J19, J20, J21, J22, J23

Commit message: terminado el diseño electrónico del grip
Parts:
- C1, C2, C3: value C -> 100nF
- RN1, RN2, RN3: value R_Network08 -> 10k
Connections:
- net +3.3V: now also C1.1, C2.1, C3.1, J1.1 (Pin_1)
- net GND: now also C1.2, C2.2, C3.2, J1.5 (Pin_5), U1.11 (DS), U1.8 (VSS), U2.8 (VSS), U3.8 (VSS)
- net LOAD: now reaches J1.2 (Pin_2)
- net LOAD: now also U1.9 (PL), U2.9 (PL), U3.9 (PL)
- net CLOCK: now reaches J1.3 (Pin_3)
- net CLOCK: now also U1.10 (CP), U2.10 (CP), U3.10 (CP)
- net DATA: now reaches J1.4 (Pin_4)
- net DATA: now also U3.3 (Q7)
- net at U2.11 (DS): now also U1.3 (Q7)
- net at U2.3 (Q7): now also U3.11 (DS)
Other:
- moved on the sheet: C1, C2, C3, J1, J10, J11, J12, J13, J14, J15, J16, J17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
